Commit message: palm frame

File: robotiq_description/urdf/robotiq_2f_85_macro.urdf.xacro (robot description, xacro)
@@ -229,4 +229,21 @@
             </inertial>
         </link>
+        <link name="${prefix}palm">
+            <visual>
+                <geometry>
+                    <box size="0.001 0.001 0.001"/>
+                </geometry>
+            </visual>
+            <collision>
+                <geometry>
+                    <box size="0.0 0.0 0.0"/>
+                </geometry>
+            </collision>
+            <inertial>
+                <origin xyz="0 0 0" rpy="0 0 0"/>
+                <mass value="0.0001"/>
+                <inertia ixx="0.0001" ixy="0" ixz="0" iyy="0.0001" iyz="0" izz="0.0001"/>
+            </inertial>
+        </link>
         <joint name="${prefix}robotiq_85_base_joint" type="fixed">
             <parent link="${parent}" />
@@ -287,4 +304,9 @@
             <mimic joint="${prefix}robotiq_85_left_knuckle_joint" />
         </joint>
+        <joint name="${prefix}palm_joint" type="fixed">
+            <parent link="${prefix}robotiq_85_base_link" />
+            <child link="${prefix}palm" />
+            <origin xyz="0 0 0.0983262" rpy="0 0 0" />
+        </joint>
     </xacro:macro>
 </robot>
