Commit message: Gazebo Classic Mimic joint plugin

File: robotiq_description/urdf/2f_85.ros2_control.xacro (robot description, xacro)
@@ -29,5 +29,5 @@
                 </xacro:if>
                 <xacro:if value="${sim_gazebo}">
-                    <plugin>ign_ros2_control/IgnitionSystem</plugin>
+                    <plugin>gazebo_ros2_control/GazeboSystem</plugin>
                 </xacro:if>
                 <xacro:if value="${use_fake_hardware}">
@@ -56,35 +56,26 @@
                 <state_interface name="velocity"/>
             </joint>
-            <!-- When simulating we need to include the rest of the gripper joints -->
+            <!-- When simulating we need to include the rest of the gripper joints.
+                 Gazebo Classic requires state interfaces so GazeboSystem registers mimic joints. -->
             <xacro:if value="${use_fake_hardware or sim_isaac or sim_gazebo}">
                 <joint name="${prefix}robotiq_85_right_knuckle_joint">
-                    <xacro:unless value="${sim_gazebo}">
-                        <state_interface name="position"/>
-                        <state_interface name="velocity"/>
-                    </xacro:unless>
+                    <state_interface name="position"/>
+                    <state_interface name="velocity"/>
                 </joint>
                 <joint name="${prefix}robotiq_85_left_inner_knuckle_joint">
-                    <xacro:unless value="${sim_gazebo}">
-                        <state_interface name="position"/>
-                        <state_interface name="velocity"/>
-                    </xacro:unless>
+                    <state_interface name="position"/>
+                    <state_interface name="velocity"/>
                 </joint>
                 <joint name="${prefix}robotiq_85_right_inner_knuckle_joint">
-                    <xacro:unless value="${sim_gazebo}">
-                        <state_interface name="position"/>
-                        <state_interface name="velocity"/>
-                    </xacro:unless>
+                    <state_interface name="position"/>
+                    <state_interface name="velocity"/>
                 </joint>
                 <joint name="${prefix}robotiq_85_left_finger_tip_joint">
-                    <xacro:unless value="${sim_gazebo}">
-                        <state_interface name="position"/>
-                        <state_interface name="velocity"/>
-                    </xacro:unless>
+                    <state_interface name="position"/>
+                    <state_interface name="velocity"/>
                 </joint>
                 <joint name="${prefix}robotiq_85_right_finger_tip_joint">
-                    <xacro:unless value="${sim_gazebo}">
-                        <state_interface name="position"/>
-                        <state_interface name="velocity"/>
-                    </xacro:unless>
+                    <state_interface name="position"/>
+                    <state_interface name="velocity"/>
                 </joint>
             </xacro:if>

File: robotiq_description/urdf/robotiq_2f_85_macro.urdf.xacro (robot description, xacro)
@@ -309,4 +309,49 @@
             <origin xyz="0 0 0.0983262" rpy="0 0 0" />
         </joint>
+        <!-- Gazebo Classic mimic joint plugins.
+             Gazebo Classic ignores URDF <mimic> tags, so we need a model plugin
+             per mimic joint to enforce the constraint in the physics engine. -->
+        <xacro:if value="${sim_gazebo}">
+            <gazebo>
+                <plugin filename="libgazebo_mimic_joint_plugin.so"
+                        name="${prefix}mimic_robotiq_85_right_knuckle">
+                    <joint>${prefix}robotiq_85_left_knuckle_joint</joint>
+                    <mimicJoint>${prefix}robotiq_85_right_knuckle_joint</mimicJoint>
+                    <multiplier>-1</multiplier>
+                </plugin>
+            </gazebo>
+            <gazebo>
+                <plugin filename="libgazebo_mimic_joint_plugin.so"
+                        name="${prefix}mimic_robotiq_85_left_inner_knuckle">
+                    <joint>${prefix}robotiq_85_left_knuckle_joint</joint>
+                    <mimicJoint>${prefix}robotiq_85_left_inner_knuckle_joint</mimicJoint>
+                    <multiplier>1</multiplier>
+                </plugin>
+            </gazebo>
+            <gazebo>
+                <plugin filename="libgazebo_mimic_joint_plugin.so"
+                        name="${prefix}mimic_robotiq_85_right_inner_knuckle">
+                    <joint>${prefix}robotiq_85_left_knuckle_joint</joint>
+                    <mimicJoint>${prefix}robotiq_85_right_inner_knuckle_joint</mimicJoint>
+                    <multiplier>-1</multiplier>
+                </plugin>
+            </gazebo>
+            <gazebo>
+                <plugin filename="libgazebo_mimic_joint_plugin.so"
+                        name="${prefix}mimic_robotiq_85_left_finger_tip">
+                    <joint>${prefix}robotiq_85_left_knuckle_joint</joint>
+                    <mimicJoint>${prefix}robotiq_85_left_finger_tip_joint</mimicJoint>
+                    <multiplier>-1</multiplier>
+                </plugin>
+            </gazebo>
+            <gazebo>
+                <plugin filename="libgazebo_mimic_joint_plugin.so"
+                        name="${prefix}mimic_robotiq_85_right_finger_tip">
+                    <joint>${prefix}robotiq_85_left_knuckle_joint</joint>
+                    <mimicJoint>${prefix}robotiq_85_right_finger_tip_joint</mimicJoint>
+                    <multiplier>1</multiplier>
+                </plugin>
+            </gazebo>
+        </xacro:if>
     </xacro:macro>
 </robot>

File: robotiq_description/urdf/robotiq_2f_85_with_adapter_macro.urdf.xacro (robot description, xacro)
@@ -19,4 +19,5 @@
         adapter_parent
         *origin
+        sim_gazebo:=false
         sim_isaac:=false
         use_fake_hardware:=false
@@ -27,5 +28,5 @@
         </xacro:robotiq_adapter>
         <xacro:robotiq_gripper name="${prefix}RobotiqGripperHardwareInterface" prefix="${prefix}" parent="${prefix}robotiq_link"
-            use_fake_hardware="${use_fake_hardware}" com_port="${com_port}" sim_isaac="${sim_isaac}" slave_address="${slave_address}">
+            use_fake_hardware="${use_fake_hardware}" com_port="${com_port}" sim_gazebo="${sim_gazebo}" sim_isaac="${sim_isaac}" slave_address="${slave_address}">
             <origin xyz="0 0 0.011" rpy="0 0 0" />
         </xacro:robotiq_gripper>
